File: eagle pcb's/avip-mod v3.sch (EAGLE design)
At the start: 44 parts, among them J1 0ohm, J2 0ohm, J3 0ohm, J4 0ohm, T1 2N2222SOT23, T2 2N2222SOT23, T3 2N2222SOT23, T4 2N2222SOT23, U1 14m2

Commit message: Fix PCB preview and update pictures
Conflict between mill and dimensions layer causing all PCB's to not show up in manufacture preview.
Add pictures of v3, v4 and v4 top PCB.
Parts:
- AVIP: value AVIP -> AVIP1.0-1.5; device XBOX:AVIP -> XBOX:AVIP1.0-1.5
- renumbered H_SYNC_IN to HS_IN, H_SYNC_OUT to HS_OUT, J4 to L1, PROG to P, RESET to R, RING to RI, SPEAK to S, TOGGLE to T, VCC2 to +, V_SYNC_IN to VS_IN, V_SYNC_OUT to VS_OUT
Connections:
- net DA: now also AVIP.6_DA; no longer AVIP.6
- net GND: now also AVIP.24_VSS; no longer AVIP.25_VDD
- net VCC: now also AVIP.1_VDD; no longer AVIP.1_VCC
