File: eagle pcb's/avip-mod v4 top.sch (EAGLE design)
At the start: 28 parts, among them J4 0ohm, U1 14m2, U2 SN74LVC2G17DBV

Commit message: Fix PCB preview and update pictures
Conflict between mill and dimensions layer causing all PCB's to not show up in manufacture preview.
Add pictures of v3, v4 and v4 top PCB.
Parts:
- renumbered H_SYNC_IN to HS_IN, H_SYNC_OUT to HS_OUT, J4 to L1, PROG to P, RESET to R, RING to RI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
